File: practice/gettingexperience/gettingexperience.kicad_pcb (KiCad board)
At the start: 2 copper layers, 283 parts, among them SW1 SW_Push, SW2 Rotary_Encoder_Switch, SW3 Rotary_Encoder_Switch, SW4 Rotary_Encoder_Switch, U1 MCP1700-3302E_SOT23, U2 SRV05-4, Y1 8MHz

Commit message: second commit
Parts:
- moved C_VDDA2 10.9 mm to (387.9, 107.7), turned to 225 degrees
- moved C_VDDA1 10.4 mm to (389.1, 108.8), turned to 225 degrees
Changed lines of the file:
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@@
   )
   (module Capacitor_SMD:C_0603_1608Metric (layer B.Cu)
-    (at 396.346748 114.569001 180)
+    (at 387.915915 107.690113 225)
     (descr "Capacitor SMD 0603 (1608 Metric), square (rectangular) end terminal, IPC_7351 nominal, (Body size source: http://www.tortai-tech.com/upload/download/2011102023233369053.pdf), generated with kicad-footprint-generator")
     (tags capacitor)
     (attr smd)
-    (fp_text reference C_VDDA2 (at 0 1.43) (layer B.SilkS)
+    (fp_text reference C_VDDA2 (at 0 1.43 45) (layer B.SilkS)
       (effects (font (size 1 1) (thickness 0.15)) (justify mirror))
     )
-    (fp_text value 1u (at 0 -1.43) (layer B.Fab)
+    (fp_text value 1u (at 0 -1.43 45) (layer B.Fab)
       (effects (font (size 1 1) (thickness 0.15)) (justify mirror))
     )
-    (fp_text user %R (at 0 0) (layer B.Fab)
+    (fp_text user %R (at 0 0 45) (layer B.Fab)
       (effects (font (size 0.4 0.4) (thickness 0.06)) (justify mirror))
     )
@@
     (fp_line (start -0.8 0.4) (end 0.8 0.4) (layer B.Fab) (width 0.1))
     (fp_line (start -0.8 -0.4) (end -0.8 0.4) (layer B.Fab) (width 0.1))
-    (pad 2 smd roundrect (at 0.7875 0 180) (size 0.875 0.95) (layers B.Cu B.Paste B.Mask) (roundrect_rratio 0.25)
+    (pad 2 smd roundrect (at 0.7875 0 225) (size 0.875 0.95) (layers B.Cu B.Paste B.Mask) (roundrect_rratio 0.25)
       (net 3 GND))
-    (pad 1 smd roundrect (at -0.7875 0 180) (size 0.875 0.95) (layers B.Cu B.Paste B.Mask) (roundrect_rratio 0.25)
+    (pad 1 smd roundrect (at -0.7875 0 225) (size 0.875 0.95) (layers B.Cu B.Paste B.Mask) (roundrect_rratio 0.25)
       (net 1 +3V3))
     (model ${KISYS3DMOD}/Capacitor_SMD.3dshapes/C_0603_1608Metric.wrl
@@
   )
   (module Capacitor_SMD:C_0603_1608Metric (layer B.Cu)
-    (at 396.367 116.205 180)
+    (at 389.087064 108.832618 225)
     (descr "Capacitor SMD 0603 (1608 Metric), square (rectangular) end terminal, IPC_7351 nominal, (Body size source: http://www.tortai-tech.com/upload/download/2011102023233369053.pdf), generated with kicad-footprint-generator")
     (tags capacitor)
     (attr smd)
-    (fp_text reference C_VDDA1 (at 0 1.43) (layer B.SilkS)
+    (fp_text reference C_VDDA1 (at 0 1.43 45) (layer B.SilkS)
       (effects (font (size 1 1) (thickness 0.15)) (justify mirror))
     )
-    (fp_text value 10u (at 0 -1.43) (layer B.Fab)
+    (fp_text value 10u (at 0 -1.43 45) (layer B.Fab)
       (effects (font (size 1 1) (thickness 0.15)) (justify mirror))
     )
-    (fp_text user %R (at 0 0) (layer B.Fab)
+    (fp_text user %R (at 0 0 45) (layer B.Fab)
       (effects (font (size 0.4 0.4) (thickness 0.06)) (justify mirror))
     )
@@
     (fp_line (start -0.8 0.4) (end 0.8 0.4) (layer B.Fab) (width 0.1))
     (fp_line (start -0.8 -0.4) (end -0.8 0.4) (layer B.Fab) (width 0.1))
-    (pad 2 smd roundrect (at 0.7875 0 180) (size 0.875 0.95) (layers B.Cu B.Paste B.Mask) (roundrect_rratio 0.25)
+    (pad 2 smd roundrect (at 0.7875 0 225) (size 0.875 0.95) (layers B.Cu B.Paste B.Mask) (roundrect_rratio 0.25)
       (net 3 GND))
-    (pad 1 smd roundrect (at -0.7875 0 180) (size 0.875 0.95) (layers B.Cu B.Paste B.Mask) (roundrect_rratio 0.25)
+    (pad 1 smd roundrect (at -0.7875 0 225) (size 0.875 0.95) (layers B.Cu B.Paste B.Mask) (roundrect_rratio 0.25)
       (net 1 +3V3))
     (model ${KISYS3DMOD}/Capacitor_SMD.3dshapes/C_0603_1608Metric.wrl

Commit message: commit for check
Parts:
- moved C_VDD3 0.84 mm to (399.3, 111.1), turned to 45 degrees
- moved R_CC2 0.13 mm to (406.3, 92.1)
- turned C_VDD1 to 135 degrees
- turned C_VDDe to 225 degrees
Other:
- net class Power added: clearance 0.2, trace_width 0.3, via_dia 0.8, via_drill 0.4
Changed lines of the file:
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@@
     (solder_mask_min_width 0.25)
     (aux_axis_origin 0 0)
-    (visible_elements FEFDF7FF)
+    (visible_elements FEFDFFFF)
     (pcbplotparams
       (layerselection 0x010fc_ffffffff)
@@
     (uvia_dia 0.3)
     (uvia_drill 0.1)
-    (add_net +3V3)
-    (add_net +5V)
     (add_net 625SPCCOL)
     (add_net 625SPCROW)
@@
     (add_net ENC3B)
     (add_net ENC3ROW)
-    (add_net GND)
     (add_net ISOENTERROW)
     (add_net ISOKEYROW)
@@
     (add_net SWDIO)
     (add_net UNSPLITROW)
+    (add_net XTAL_IN)
+    (add_net XTAL_OUT)
+  )
+  (net_class Power ""
+    (clearance 0.2)
+    (trace_width 0.3)
+    (via_dia 0.8)
+    (via_drill 0.4)
+    (uvia_dia 0.3)
+    (uvia_drill 0.1)
+    (add_net +3V3)
+    (add_net +5V)
+    (add_net GND)
     (add_net USB_D+)
     (add_net USB_D-)
     (add_net VCC)
-    (add_net XTAL_IN)
-    (add_net XTAL_OUT)
   )
   (module MX_Only:MXOnly-1.25U-NoLED (layer F.Cu)
@@
   )
   (module Resistor_SMD:R_0603_1608Metric (layer B.Cu)
-    (at 406.4 92.1005 90)
+    (at 406.273 92.1005 90)
     (descr "Resistor SMD 0603 (1608 Metric), square (rectangular) end terminal, IPC_7351 nominal, (Body size source: http://www.tortai-tech.com/upload/download/2011102023233369053.pdf), generated with kicad-footprint-generator")
     (tags resistor)
@@
   )
   (module Capacitor_SMD:C_0603_1608Metric (layer B.Cu)
-    (at 398.907 111.887 225)
+    (at 399.25625 111.125 45)
     (descr "Capacitor SMD 0603 (1608 Metric), square (rectangular) end terminal, IPC_7351 nominal, (Body size source: http://www.tortai-tech.com/upload/download/2011102023233369053.pdf), generated with kicad-footprint-generator")
     (tags capacitor)
@@
     (fp_line (start -0.8 0.4) (end 0.8 0.4) (layer B.Fab) (width 0.1))
     (fp_line (start -0.8 -0.4) (end -0.8 0.4) (layer B.Fab) (width 0.1))
-    (pad 2 smd roundrect (at 0.7875 0 225) (size 0.875 0.95) (layers B.Cu B.Paste B.Mask) (roundrect_rratio 0.25)
+    (pad 2 smd roundrect (at 0.7875 0 45) (size 0.875 0.95) (layers B.Cu B.Paste B.Mask) (roundrect_rratio 0.25)
       (net 3 GND))
-    (pad 1 smd roundrect (at -0.7875 0 225) (size 0.875 0.95) (layers B.Cu B.Paste B.Mask) (roundrect_rratio 0.25)
+    (pad 1 smd roundrect (at -0.7875 0 45) (size 0.875 0.95) (layers B.Cu B.Paste B.Mask) (roundrect_rratio 0.25)
       (net 1 +3V3))
     (model ${KISYS3DMOD}/Capacitor_SMD.3dshapes/C_0603_1608Metric.wrl
@@
   )
   (module Capacitor_SMD:C_0603_1608Metric (layer B.Cu)
-    (at 392.049 92.964 135)
+    (at 392.049 92.964 225)
     (descr "Capacitor SMD 0603 (1608 Metric), square (rectangular) end terminal, IPC_7351 nominal, (Body size source: http://www.tortai-tech.com/upload/download/2011102023233369053.pdf), generated with kicad-footprint-generator")
     (tags capacitor)
     (attr smd)
-    (fp_text reference C_VDDe (at 0 1.43 135) (layer B.SilkS)
+    (fp_text reference C_VDDe (at 0 1.43 45) (layer B.SilkS)
       (effects (font (size 1 1) (thickness 0.15)) (justify mirror))
     )
-    (fp_text value 100n (at 0 -1.43 135) (layer B.Fab)
+    (fp_text value 100n (at 0 -1.43 45) (layer B.Fab)
       (effects (font (size 1 1) (thickness 0.15)) (justify mirror))
     )
-    (fp_text user %R (at 0 0 135) (layer B.Fab)
+    (fp_text user %R (at 0 0 45) (layer B.Fab)
       (effects (font (size 0.4 0.4) (thickness 0.06)) (justify mirror))
     )
@@
     (fp_line (start -0.8 0.4) (end 0.8 0.4) (layer B.Fab) (width 0.1))
     (fp_line (start -0.8 -0.4) (end -0.8 0.4) (layer B.Fab) (width 0.1))
-    (pad 2 smd roundrect (at 0.7875 0 135) (size 0.875 0.95) (layers B.Cu B.Paste B.Mask) (roundrect_rratio 0.25)
+    (pad 2 smd roundrect (at 0.7875 0 225) (size 0.875 0.95) (layers B.Cu B.Paste B.Mask) (roundrect_rratio 0.25)
       (net 3 GND))
-    (pad 1 smd roundrect (at -0.7875 0 135) (size 0.875 0.95) (layers B.Cu B.Paste B.Mask) (roundrect_rratio 0.25)
+    (pad 1 smd roundrect (at -0.7875 0 225) (size 0.875 0.95) (layers B.Cu B.Paste B.Mask) (roundrect_rratio 0.25)
       (net 1 +3V3))
     (model ${KISYS3DMOD}/Capacitor_SMD.3dshapes/C_0603_1608Metric.wrl
@@
   )
   (module Capacitor_SMD:C_0603_1608Metric (layer B.Cu)
-    (at 405.13 98.298 45)
+    (at 405.13 98.298 135)
     (descr "Capacitor SMD 0603 (1608 Metric), square (rectangular) end terminal, IPC_7351 nominal, (Body size source: http://www.tortai-tech.com/upload/download/2011102023233369053.pdf), generated with kicad-footprint-generator")
     (tags capacitor)
     (attr smd)
-    (fp_text reference C_VDD1 (at 0 1.43 45) (layer B.SilkS)
+    (fp_text reference C_VDD1 (at 0 1.43 135) (layer B.SilkS)
       (effects (font (size 1 1) (thickness 0.15)) (justify mirror))
     )
-    (fp_text value 100n (at 0 -1.43 45) (layer B.Fab)
+    (fp_text value 100n (at 0 -1.43 135) (layer B.Fab)
       (effects (font (size 1 1) (thickness 0.15)) (justify mirror))
     )
-    (fp_text user %R (at 0 0 45) (layer B.Fab)
+    (fp_text user %R (at 0 0 135) (layer B.Fab)
       (effects (font (size 0.4 0.4) (thickness 0.06)) (justify mirror))
     )
@@
     (fp_line (start -0.8 0.4) (end 0.8 0.4) (layer B.Fab) (width 0.1))
     (fp_line (start -0.8 -0.4) (end -0.8 0.4) (layer B.Fab) (width 0.1))
-    (pad 2 smd roundrect (at 0.7875 0 45) (size 0.875 0.95) (layers B.Cu B.Paste B.Mask) (roundrect_rratio 0.25)
+    (pad 2 smd roundrect (at 0.7875 0 135) (size 0.875 0.95) (layers B.Cu B.Paste B.Mask) (roundrect_rratio 0.25)
       (net 3 GND))
-    (pad 1 smd roundrect (at -0.7875 0 45) (size 0.875 0.95) (layers B.Cu B.Paste B.Mask) (roundrect_rratio 0.25)
+    (pad 1 smd roundrect (at -0.7875 0 135) (size 0.875 0.95) (layers B.Cu B.Paste B.Mask) (roundrect_rratio 0.25)
       (net 1 +3V3))
     (model ${KISYS3DMOD}/Capacitor_SMD.3dshapes/C_0603_1608Metric.wrl
