File: practice/gettingexperience/gettingexperience.sch (KiCad schematic (older format))
At the start: 283 parts, among them SW1 SW_Push, SW2 Rotary_Encoder_Switch, SW3 Rotary_Encoder_Switch, SW4 Rotary_Encoder_Switch, U1 MCP1700-3302E_SOT23, U2 SRV05-4, U3 STM32F303RCTx, Y1 8MHz

Commit message: second commit
Parts:
- removed JBREAKOUT1: Conn_01x08_Male, Connector_PinHeader_2.54mm:PinHeader_1x08_P2.54mm_Vertical, symbol Connector:Conn_01x08_Male
- added C_RESET1: 100nF, symbol Device:C_Small
- R_USB1: value 5.1k -> 1.5k
Connections:
- net BREAKOUT1 is gone; now on net LEDSTAT1: U3.58 (PB6)
- net BREAKOUT2 is gone; now on net LEDSTAT2: U3.59 (PB7)
- net BREAKOUT3 is gone; now on net LEDSTAT3: U3.61 (PB8)
- net COL11: now also U3.16 (PA2); no longer U3.15 (PA1)
- net COL12: now also U3.17 (PA3); no longer U3.16 (PA2)
- net COL13: now also U3.20 (PA4); no longer U3.17 (PA3)
- net COL14: now also U3.21 (PA5); no longer U3.20 (PA4)
- net COL15: now also U3.22 (PA6); no longer U3.21 (PA5)
- net COL16: now also U3.23 (PA7); no longer U3.22 (PA6)
- net COL17: now also U3.41 (PA8); no longer U3.23 (PA7)
- net COL18: now also U3.42 (PA9); no longer U3.41 (PA8)
- net GND: now also C_RESET1.1
- net LEDSTAT1: no longer U3.42 (PA9)
- net LEDSTAT2: no longer U3.43 (PA10)
- net LEDSTAT3: no longer U3.50 (PA15)
- net NRST: now also C_RESET1.2
- net RGB: now also U3.15 (PA1); no longer U3.36 (PB15)
- net BREAKOUT4: no longer names the net of U3.62 (PB9)
- net BREAKOUT5: no longer names the net of U3.29 (PB10)
- net BREAKOUT6: no longer names the net of U3.30 (PB11)
- net BREAKOUT7: no longer names the net of U3.33 (PB12)
- net BREAKOUT8: no longer names the net of U3.35 (PB14)
- no-connect marks 9 -> 8
Other:
- moved on the sheet: R_RGB1
Changed lines of the file:
@@
 EELAYER 30 0
 EELAYER END
-$Descr A4 11693 8268
+$Descr A3 16535 11693
 encoding utf-8
 Sheet 1 1
@@
 	10050 5200 9950 5200
 Wire Wire Line
-	9250 5200 9550 5200
+	9250 5200 9450 5200
 Text GLabel 9500 4550 0    50   Input ~ 0
 BOOT0
@@
 Text GLabel 200  12650 0    39   Input ~ 0
 ROW5
-$Comp
-L Connector:Conn_01x08_Male JBREAKOUT1
-U 1 1 60B24F91
-P 6000 6150
-F 0 "JBREAKOUT1" H 6108 6631 50  0000 C CNN
-F 1 "Conn_01x08_Male" H 6108 6540 50  0000 C CNN
-F 2 "Connector_PinHeader_2.54mm:PinHeader_1x08_P2.54mm_Vertical" H 6000 6150 50  0001 C CNN
-F 3 "~" H 6000 6150 50  0001 C CNN
-	1    6000 6150
-	1    0    0    -1
-$EndComp
-Text GLabel 6200 5850 2    39   Input ~ 0
-BREAKOUT1
-Text GLabel 6200 5950 2    39   Input ~ 0
-BREAKOUT2
-Text GLabel 6200 6050 2    39   Input ~ 0
-BREAKOUT3
-Text GLabel 6200 6150 2    39   Input ~ 0
-BREAKOUT4
-Text GLabel 6200 6250 2    39   Input ~ 0
-BREAKOUT5
-Text GLabel 6200 6350 2    39   Input ~ 0
-BREAKOUT6
-Text GLabel 6200 6450 2    39   Input ~ 0
-BREAKOUT7
-Text GLabel 6200 6550 2    39   Input ~ 0
-BREAKOUT8
 Text GLabel 13850 2300 2    50   Input ~ 0
 SWDIO
 Text GLabel 13850 2400 2    50   Input ~ 0
 SWCLK
-$Comp
-L MCU_ST_STM32F3:STM32F303RCTx U3
-U 1 1 60389791
-P 13150 2600
-F 0 "U3" H 13150 1400 50  0000 C CNN
-F 1 "STM32F303RCTx" H 13150 1300 50  0000 C CNN
-F 2 "Package_QFP:LQFP-64_10x10mm_P0.5mm" H 12550 900 50  0001 R CNN
-F 3 "http://www.st.com/st-web-ui/static/active/en/resource/technical/document/datasheet/DM00058181.pdf" H 13150 2600 50  0001 C CNN
-	1    13150 2600
-	1    0    0    -1
-$EndComp
-Wire Wire Line
-	13350 4400 13250 4400
 Wire Wire Line
 	13050 4400 13050 4500
-Connection ~ 13050 4400
-Connection ~ 13150 4400
-Wire Wire Line
-	13150 4400 13050 4400
-Connection ~ 13250 4400
-Wire Wire Line
-	13250 4400 13150 4400
 $Comp
 L power:GND #PWR036
@@
 $EndComp
 Wire Wire Line
-	13450 800  13350 800
-Connection ~ 13050 800
-Wire Wire Line
-	13050 800  12950 800
-Connection ~ 13150 800
-Wire Wire Line
-	13150 800  13050 800
-Connection ~ 13250 800
-Wire Wire Line
-	13250 800  13150 800
-Connection ~ 13350 800
-Wire Wire Line
-	13350 800  13250 800
-Wire Wire Line
 	12950 800  12950 700
-Connection ~ 12950 800
 $Comp
 L power:+3.3V #PWR01
@@
 P 14450 2000
 F 0 "R_USB1" H 14509 2046 50  0000 L CNN
-F 1 "5.1k" H 14509 1955 50  0000 L CNN
+F 1 "1.5k" H 14509 1955 50  0000 L CNN
 F 2 "Resistor_SMD:R_0603_1608Metric" H 14450 2000 50  0001 C CNN
 F 3 "~" H 14450 2000 50  0001 C CNN
@@
 	1    0    0    -1
 $EndComp
-Text GLabel 13850 1800 2    39   Input ~ 0
+Text GLabel 13850 1900 2    39   Input ~ 0
 COL18
-Text GLabel 13850 1700 2    39   Input ~ 0
+Text GLabel 13850 1800 2    39   Input ~ 0
 COL17
-Text GLabel 13850 1600 2    39   Input ~ 0
+Text GLabel 13850 1700 2    39   Input ~ 0
 COL16
-Text GLabel 13850 1500 2    39   Input ~ 0
+Text GLabel 13850 1600 2    39   Input ~ 0
 COL15
-Text GLabel 13850 1400 2    39   Input ~ 0
+Text GLabel 13850 1500 2    39   Input ~ 0
 COL14
-Text GLabel 13850 1300 2    39   Input ~ 0
+Text GLabel 13850 1400 2    39   Input ~ 0
 COL13
-Text GLabel 13850 1200 2    39   Input ~ 0
+Text GLabel 13850 1300 2    39   Input ~ 0
 COL12
-Text GLabel 13850 1100 2    39   Input ~ 0
+Text GLabel 13850 1200 2    39   Input ~ 0
 COL11
 Text GLabel 13850 1000 2    39   Input ~ 0
@@
 	14450 1900 14450 1800
 $Comp
-L Device:R_Small R_RGB1
-U 1 1 608679FF
-P 14450 4300
-F 0 "R_RGB1" H 14391 4254 50  0000 R CNN
-F 1 "10k" H 14391 4345 50  0000 R CNN
-F 2 "Resistor_SMD:R_0603_1608Metric" H 14450 4300 50  0001 C CNN
-F 3 "~" H 14450 4300 50  0001 C CNN
-	1    14450 4300
-	1    0    0    -1
-$EndComp
-$Comp
 L power:+5V #PWR034
 U 1 1 60867A05
-P 14450 4400
-F 0 "#PWR034" H 14450 4250 50  0001 C CNN
-F 1 "+5V" H 14465 4573 50  0000 C CNN
-F 2 "" H 14450 4400 50  0001 C CNN
-F 3 "" H 14450 4400 50  0001 C CNN
-	1    14450 4400
+P 14550 1300
+F 0 "#PWR034" H 14550 1150 50  0001 C CNN
+F 1 "+5V" H 14565 1473 50  0000 C CNN
+F 2 "" H 14550 1300 50  0001 C CNN
+F 3 "" H 14550 1300 50  0001 C CNN
+	1    14550 1300
 	-1   0    0    1
 $EndComp
-Wire Wire Line
-	14450 4200 13850 4200
-Wire Wire Line
-	14450 4200 14600 4200
-Connection ~ 14450 4200
-Text GLabel 14600 4200 2    50   Input ~ 0
+Text GLabel 14700 1100 2    50   Input ~ 0
 RGB
 Text GLabel 12450 4000 0    39   Input ~ 0
@@
 Text GLabel 12450 4100 0    39   Input ~ 0
 COL8
-Text GLabel 13850 2000 2    50   Input ~ 0
+Text GLabel 13850 3400 2    50   Input ~ 0
 LEDSTAT2
-Text GLabel 13850 1900 2    50   Input ~ 0
+Text GLabel 13850 3300 2    50   Input ~ 0
 LEDSTAT1
-Text GLabel 13850 2500 2    50   Input ~ 0
+Text GLabel 13850 3500 2    50   Input ~ 0
 LEDSTAT3
 Text GLabel 13850 2700 2    39   Input ~ 0
@@
 Text GLabel 13850 3000 2    39   Input ~ 0
 ROW3
-NoConn ~ 13850 4000
 Text GLabel 13850 3100 2    39   Input ~ 0
 ROW4
 Text GLabel 13850 3200 2    39   Input ~ 0
 ROW5
-Text GLabel 13850 3300 2    39   Input ~ 0
-BREAKOUT1
-Text GLabel 13850 3400 2    39   Input ~ 0
-BREAKOUT2
-Text GLabel 13850 3500 2    39   Input ~ 0
-BREAKOUT3
-Text GLabel 13850 3600 2    39   Input ~ 0
-BREAKOUT4
-Text GLabel 13850 3700 2    39   Input ~ 0
-BREAKOUT5
-Text GLabel 13850 3800 2    39   Input ~ 0
-BREAKOUT6
-Text GLabel 13850 3900 2    39   Input ~ 0
-BREAKOUT7
-Text GLabel 13850 4100 2    39   Input ~ 0
-BREAKOUT8
 NoConn ~ 12450 2300
 NoConn ~ 12450 2500
@@
 Wire Wire Line
 	9750 10050 9750 11550
+Wire Wire Line
+	13350 4400 13250 4400
+Connection ~ 13250 4400
+Wire Wire Line
+	13250 4400 13150 4400
+Wire Wire Line
+	13150 4400 13050 4400
+Connection ~ 13150 4400
+Connection ~ 13050 4400
+Wire Wire Line
+	13450 800  13350 800
+Connection ~ 13350 800
+Wire Wire Line
+	13350 800  13250 800
+Connection ~ 13250 800
+Wire Wire Line
+	13250 800  13150 800
+Connection ~ 13150 800
+Wire Wire Line
+	13150 800  13050 800
+Wire Wire Line
+	13050 800  12950 800
+Connection ~ 13050 800
+Connection ~ 12950 800
+$Comp
+L MCU_ST_STM32F3:STM32F303RCTx U3
+U 1 1 60389791
+P 13150 2600
+F 0 "U3" H 13150 1400 50  0000 C CNN
+F 1 "STM32F303RCTx" H 13150 1300 50  0000 C CNN
+F 2 "Package_QFP:LQFP-64_10x10mm_P0.5mm" H 12550 900 50  0001 R CNN
+F 3 "http://www.st.com/st-web-ui/static/active/en/resource/technical/document/datasheet/DM00058181.pdf" H 13150 2600 50  0001 C CNN
+	1    13150 2600
+	1    0    0    -1
+$EndComp
+$Comp
+L Device:C_Small C_RESET1
+U 1 1 5FCA4C3C
+P 9750 5400
+F 0 "C_RESET1" V 9521 5400 50  0000 C CNN
+F 1 "100nF" V 9612 5400 50  0000 C CNN
+F 2 "" H 9750 5400 50  0001 C CNN
+F 3 "~" H 9750 5400 50  0001 C CNN
+	1    9750 5400
+	0    1    1    0
+$EndComp
+Wire Wire Line
+	9450 5200 9450 5400
+Wire Wire Line
+	9450 5400 9650 5400
+Connection ~ 9450 5200
+Wire Wire Line
+	9450 5200 9550 5200
+Wire Wire Line
+	9850 5400 9950 5400
+Wire Wire Line
+	9950 5400 9950 5200
+Connection ~ 9950 5200
+Connection ~ 14550 1100
+Wire Wire Line
+	13850 1100 14550 1100
+Wire Wire Line
+	14550 1100 14700 1100
+$Comp
+L Device:R_Small R_RGB1
+U 1 1 608679FF
+P 14550 1200
+F 0 "R_RGB1" H 14491 1154 50  0000 R CNN
+F 1 "10k" H 14491 1245 50  0000 R CNN
+F 2 "Resistor_SMD:R_0603_1608Metric" H 14550 1200 50  0001 C CNN
+F 3 "~" H 14550 1200 50  0001 C CNN
+	1    14550 1200
+	1    0    0    -1
+$EndComp
 $EndSCHEMATC

Commit message: commit for check
Connections:
- net COL11: now also U3.15 (PA1); no longer U3.16 (PA2)
- net COL12: now also U3.16 (PA2); no longer U3.17 (PA3)
- net COL13: now also U3.17 (PA3); no longer U3.20 (PA4)
- net COL14: now also U3.20 (PA4); no longer U3.21 (PA5)
- net COL15: now also U3.23 (PA7); no longer U3.22 (PA6)
- net COL16: now also U3.41 (PA8); no longer U3.23 (PA7)
- net COL17: now also U3.42 (PA9); no longer U3.41 (PA8)
- net COL18: now also U3.43 (PA10); no longer U3.42 (PA9)
- net RGB: now also U3.57 (PB5); no longer U3.15 (PA1)
- net ROW5: now also U3.62 (PB9); no longer U3.57 (PB5)
- no-connect marks 8 -> 10
Other:
- moved on the sheet: R_RGB1
Changed lines of the file:
@@
 	1    0    0    -1
 $EndComp
+Text GLabel 13850 2000 2    39   Input ~ 0
+COL18
 Text GLabel 13850 1900 2    39   Input ~ 0
-COL18
+COL17
 Text GLabel 13850 1800 2    39   Input ~ 0
-COL17
+COL16
 Text GLabel 13850 1700 2    39   Input ~ 0
-COL16
-Text GLabel 13850 1600 2    39   Input ~ 0
 COL15
-Text GLabel 13850 1500 2    39   Input ~ 0
+Text GLabel 13850 1400 2    39   Input ~ 0
 COL14
-Text GLabel 13850 1400 2    39   Input ~ 0
+Text GLabel 13850 1300 2    39   Input ~ 0
 COL13
-Text GLabel 13850 1300 2    39   Input ~ 0
+Text GLabel 13850 1200 2    39   Input ~ 0
 COL12
-Text GLabel 13850 1200 2    39   Input ~ 0
+Text GLabel 13850 1100 2    39   Input ~ 0
 COL11
 Text GLabel 13850 1000 2    39   Input ~ 0
@@
 L power:+5V #PWR034
 U 1 1 60867A05
-P 14550 1300
-F 0 "#PWR034" H 14550 1150 50  0001 C CNN
-F 1 "+5V" H 14565 1473 50  0000 C CNN
-F 2 "" H 14550 1300 50  0001 C CNN
-F 3 "" H 14550 1300 50  0001 C CNN
-	1    14550 1300
+P 14550 3400
+F 0 "#PWR034" H 14550 3250 50  0001 C CNN
+F 1 "+5V" H 14565 3573 50  0000 C CNN
+F 2 "" H 14550 3400 50  0001 C CNN
+F 3 "" H 14550 3400 50  0001 C CNN
+	1    14550 3400
 	-1   0    0    1
 $EndComp
-Text GLabel 14700 1100 2    50   Input ~ 0
+Text GLabel 14700 3200 2    50   Input ~ 0
 RGB
 Text GLabel 12450 4000 0    39   Input ~ 0
@@
 Text GLabel 13850 3100 2    39   Input ~ 0
 ROW4
-Text GLabel 13850 3200 2    39   Input ~ 0
+Text GLabel 13850 3600 2    39   Input ~ 0
 ROW5
 NoConn ~ 12450 2300
@@
 	9950 5400 9950 5200
 Connection ~ 9950 5200
-Connection ~ 14550 1100
-Wire Wire Line
-	13850 1100 14550 1100
-Wire Wire Line
-	14550 1100 14700 1100
+Connection ~ 14550 3200
+Wire Wire Line
+	13850 3200 14550 3200
+Wire Wire Line
+	14550 3200 14700 3200
 $Comp
 L Device:R_Small R_RGB1
 U 1 1 608679FF
-P 14550 1200
-F 0 "R_RGB1" H 14491 1154 50  0000 R CNN
-F 1 "10k" H 14491 1245 50  0000 R CNN
-F 2 "Resistor_SMD:R_0603_1608Metric" H 14550 1200 50  0001 C CNN
-F 3 "~" H 14550 1200 50  0001 C CNN
-	1    14550 1200
-	1    0    0    -1
-$EndComp
+P 14550 3300
+F 0 "R_RGB1" H 14491 3254 50  0000 R CNN
+F 1 "10k" H 14491 3345 50  0000 R CNN
+F 2 "Resistor_SMD:R_0603_1608Metric" H 14550 3300 50  0001 C CNN
+F 3 "~" H 14550 3300 50  0001 C CNN
+	1    14550 3300
+	1    0    0    -1
+$EndComp
+NoConn ~ 13850 1500
+NoConn ~ 13850 1600
 $EndSCHEMATC
